File: hw/R2P_PS_module.brd (EAGLE design)
At the start: 40 x 60 mm, 67 parts, among them U1 STM32F103CX, U4 TPS5450, U5 LD3985XX, X2 OSC-XTAL212M_

Commit message: Added R2 value
Parts:
- R2: value (none) -> 4k7

Commit message: added missing component values
Parts:
- C1: value 10nF -> 100nF
- R3: value (none) -> 100
Changed lines of the file:
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@@
 <element name="R7" library="rcl" package="R0603" value="1k" x="36.03625" y="35.2425" rot="R270"/>
 <element name="D4" library="dp_devices" package="SOD-323F" value="" x="34.13125" y="35.2425" rot="R90"/>
-<element name="R3" library="rcl" package="R0603" value="" x="27.46375" y="38.4175" rot="R270"/>
-<element name="C1" library="rcl" package="C0603" value="10nF" x="29.5275" y="38.4175" rot="R270"/>
+<element name="R3" library="rcl" package="R0603" value="100" x="27.46375" y="38.4175" rot="R270"/>
+<element name="C1" library="rcl" package="C0603" value="100nF" x="29.5275" y="38.4175" rot="R270"/>
 <element name="C8" library="rcl" package="E5-10,5" value="" x="6.6675" y="28.2575" rot="R90"/>
 <element name="C13" library="rcl" package="E5-10,5" value="100uF 50V" x="18.7325" y="37.1475" rot="R270"/>
